File: KiCad project/Sheet1.sch (KiCad schematic (older format))
At the start: 33 parts, among them CON1 USB-MICRO-B, U1 EFM32GG332, U2 BQ25011, U3 BQ27421-G1, U4 IP4220CZ6

Commit message: PCB finalised, Gerbers created for v0.5
New footprints, fixes in schematic, PCB final design, plotted Gerbers
for prototype production
Parts:
- removed TP12, TP13, TP14, TP15, TP16: TESTPAD, Anastasia:Test_Point_Round-SMD-Pad, symbol TESTPAD
- R3: value 1K6 -> 4K7
Connections:
- wire segments 99 -> 96
Changed lines of the file:
@@
 $Descr A4 11693 8268
 encoding utf-8
-Sheet 2 10
+Sheet 10 10
 Title "Power"
 Date "14 March 2015"
@@
 $EndComp
 $Comp
-L GND #PWR01
+L GND #PWR045
 U 1 1 55047461
 P 2250 1400
-F 0 "#PWR01" H 2250 1150 60  0001 C CNN
+F 0 "#PWR045" H 2250 1150 60  0001 C CNN
 F 1 "GND" H 2250 1250 60  0000 C CNN
 F 2 "" H 2250 1400 60  0000 C CNN
@@
 $EndComp
 $Comp
-L +3V3 #PWR02
+L +3V3 #PWR046
 U 1 1 5504746F
 P 2050 1950
-F 0 "#PWR02" H 2050 1800 60  0001 C CNN
+F 0 "#PWR046" H 2050 1800 60  0001 C CNN
 F 1 "+3V3" H 2050 2090 60  0000 C CNN
 F 2 "" H 2050 1950 60  0000 C CNN
@@
 $EndComp
 $Comp
-L GND #PWR03
+L GND #PWR047
 U 1 1 55047491
 P 2750 2650
-F 0 "#PWR03" H 2750 2400 60  0001 C CNN
+F 0 "#PWR047" H 2750 2400 60  0001 C CNN
 F 1 "GND" H 2750 2500 60  0000 C CNN
 F 2 "" H 2750 2650 60  0000 C CNN
@@
 $EndComp
 $Comp
-L GND #PWR04
+L GND #PWR048
 U 1 1 5504749E
 P 6250 1650
-F 0 "#PWR04" H 6250 1400 60  0001 C CNN
+F 0 "#PWR048" H 6250 1400 60  0001 C CNN
 F 1 "GND" H 6250 1500 60  0000 C CNN
 F 2 "" H 6250 1650 60  0000 C CNN
@@
 $EndComp
 $Comp
-L +3V3 #PWR05
+L +3V3 #PWR049
 U 1 1 550474A4
 P 6950 2250
-F 0 "#PWR05" H 6950 2100 60  0001 C CNN
+F 0 "#PWR049" H 6950 2100 60  0001 C CNN
 F 1 "+3V3" H 6950 2390 60  0000 C CNN
 F 2 "" H 6950 2250 60  0000 C CNN
@@
 $EndComp
 $Comp
-L GND #PWR06
+L GND #PWR050
 U 1 1 550474AB
 P 6850 2750
-F 0 "#PWR06" H 6850 2500 60  0001 C CNN
+F 0 "#PWR050" H 6850 2500 60  0001 C CNN
 F 1 "GND" H 6850 2600 60  0000 C CNN
 F 2 "" H 6850 2750 60  0000 C CNN
@@
 $EndComp
 $Comp
-L GND #PWR07
+L GND #PWR051
 U 1 1 550474DE
 P 2300 3750
-F 0 "#PWR07" H 2300 3500 60  0001 C CNN
+F 0 "#PWR051" H 2300 3500 60  0001 C CNN
 F 1 "GND" H 2300 3600 60  0000 C CNN
 F 2 "" H 2300 3750 60  0000 C CNN
@@
 $EndComp
 $Comp
-L GND #PWR08
+L GND #PWR052
 U 1 1 550474EB
 P 2250 5400
-F 0 "#PWR08" H 2250 5150 60  0001 C CNN
+F 0 "#PWR052" H 2250 5150 60  0001 C CNN
 F 1 "GND" H 2250 5250 60  0000 C CNN
 F 2 "" H 2250 5400 60  0000 C CNN
@@
 $EndComp
 $Comp
-L GND #PWR09
+L GND #PWR053
 U 1 1 55047506
 P 4700 4100
-F 0 "#PWR09" H 4700 3850 60  0001 C CNN
+F 0 "#PWR053" H 4700 3850 60  0001 C CNN
 F 1 "GND" H 4700 3950 60  0000 C CNN
 F 2 "" H 4700 4100 60  0000 C CNN
@@
 $EndComp
 $Comp
-L +3V3 #PWR010
+L +3V3 #PWR054
 U 1 1 5504750C
 P 4700 3450
-F 0 "#PWR010" H 4700 3300 60  0001 C CNN
+F 0 "#PWR054" H 4700 3300 60  0001 C CNN
 F 1 "+3V3" H 4700 3590 60  0000 C CNN
 F 2 "" H 4700 3450 60  0000 C CNN
@@
 P 4100 4150
 F 0 "R3" V 4180 4150 50  0000 C CNN
-F 1 "1K6" V 4107 4151 50  0000 C CNN
+F 1 "4K7" V 4107 4151 50  0000 C CNN
 F 2 "Resistors_SMD:R_0603" V 4030 4150 30  0001 C CNN
 F 3 "" H 4100 4150 30  0000 C CNN
@@
 $EndComp
 $Comp
-L GND #PWR011
+L GND #PWR055
 U 1 1 5504752A
 P 2950 1850
-F 0 "#PWR011" H 2950 1600 60  0001 C CNN
+F 0 "#PWR055" H 2950 1600 60  0001 C CNN
 F 1 "GND" H 2950 1700 60  0000 C CNN
 F 2 "" H 2950 1850 60  0000 C CNN
@@
 $EndComp
 $Comp
-L GND #PWR012
+L GND #PWR056
 U 1 1 55047918
 P 8250 5800
-F 0 "#PWR012" H 8250 5550 60  0001 C CNN
+F 0 "#PWR056" H 8250 5550 60  0001 C CNN
 F 1 "GND" H 8250 5650 60  0000 C CNN
 F 2 "" H 8250 5800 60  0000 C CNN
@@
 Text HLabel 1750 1000 0    60   Input ~ 0
 MCU_RESET
-$Comp
-L TESTPAD TP12
-U 1 1 5506D7F2
-P 1750 1150
-F 0 "TP12" H 2000 1150 60  0000 C CNN
-F 1 "TESTPAD" H 1800 950 60  0001 C CNN
-F 2 "Anastasia:Test_Point_Round-SMD-Pad" H 2000 1150 60  0001 C CNN
-F 3 "" H 2000 1150 60  0000 C CNN
-	1    1750 1150
-	-1   0    0    -1
-$EndComp
 NoConn ~ 2600 3550
 NoConn ~ 3700 4350
@@
 $EndComp
 $Comp
-L +3V3 #PWR013
+L +3V3 #PWR057
 U 1 1 55072596
 P 1700 3600
-F 0 "#PWR013" H 1700 3450 60  0001 C CNN
+F 0 "#PWR057" H 1700 3450 60  0001 C CNN
 F 1 "+3V3" H 1700 3740 60  0000 C CNN
 F 2 "" H 1700 3600 60  0000 C CNN
@@
 	1    1700 3600
 	1    0    0    -1
-$EndComp
-$Comp
-L TESTPAD TP14
-U 1 1 55072D4F
-P 1650 4600
-F 0 "TP14" H 1900 4600 60  0000 C CNN
-F 1 "TESTPAD" H 1700 4400 60  0001 C CNN
-F 2 "Anastasia:Test_Point_Round-SMD-Pad" H 1900 4600 60  0001 C CNN
-F 3 "" H 1900 4600 60  0000 C CNN
-	1    1650 4600
-	-1   0    0    -1
-$EndComp
-$Comp
-L TESTPAD TP15
-U 1 1 550731F6
-P 1650 5500
-F 0 "TP15" H 1900 5500 60  0000 C CNN
-F 1 "TESTPAD" H 1700 5300 60  0001 C CNN
-F 2 "Anastasia:Test_Point_Round-SMD-Pad" H 1900 5500 60  0001 C CNN
-F 3 "" H 1900 5500 60  0000 C CNN
-	1    1650 5500
-	-1   0    0    -1
 $EndComp
 NoConn ~ 2650 5100
@@
 $EndComp
 $Comp
-L GND #PWR014
+L GND #PWR058
 U 1 1 55085BD1
 P 6250 6200
-F 0 "#PWR014" H 6250 5950 60  0001 C CNN
+F 0 "#PWR058" H 6250 5950 60  0001 C CNN
 F 1 "GND" H 6250 6050 60  0000 C CNN
 F 2 "" H 6250 6200 60  0000 C CNN
@@
 $EndComp
 $Comp
-L GND #PWR015
+L GND #PWR059
 U 1 1 55086166
 P 4400 5850
-F 0 "#PWR015" H 4400 5600 60  0001 C CNN
+F 0 "#PWR059" H 4400 5600 60  0001 C CNN
 F 1 "GND" H 4400 5700 60  0000 C CNN
 F 2 "" H 4400 5850 60  0000 C CNN
@@
 Wire Wire Line
 	3800 3850 3700 3850
-Connection ~ 1650 5400
-Wire Wire Line
-	1650 4800 1650 4600
 Wire Wire Line
 	1700 3700 1700 3600
@@
 Wire Wire Line
 	3700 4250 3900 4250
-Connection ~ 1900 1000
-Wire Wire Line
-	1900 1150 1900 1000
-Wire Wire Line
-	1750 1150 1900 1150
 Connection ~ 7400 5800
 Connection ~ 7250 5800
@@
 Connection ~ 2250 1000
 Connection ~ 2250 1400
-Connection ~ 1750 1000
 Wire Wire Line
 	3750 2150 3750 2050
@@
 	3200 1850 2950 1850
 Wire Wire Line
-	1650 5200 1650 5500
+	1650 5400 1650 5200
 Wire Wire Line
 	2650 5400 2650 5200
@@
 	2250 6550 2000 6550
 $Comp
-L GND #PWR016
+L GND #PWR060
 U 1 1 550950F7
 P 650 6550
-F 0 "#PWR016" H 650 6300 60  0001 C CNN
+F 0 "#PWR060" H 650 6300 60  0001 C CNN
 F 1 "GND" H 650 6400 60  0000 C CNN
 F 2 "" H 650 6550 60  0000 C CNN
@@
 	2050 5000 2050 5750
 Wire Wire Line
-	2000 6450 2000 6000
-Connection ~ 2000 6000
-Wire Wire Line
 	2000 6650 2150 6650
-Wire Wire Line
-	2150 6650 2150 5750
-Connection ~ 2150 5750
 Text Notes 1150 6950 0    60   ~ 0
 ESD Protection\n
@@
 Wire Wire Line
 	6100 5150 6100 5600
-$Comp
-L TESTPAD TP16
-U 1 1 550C93EA
-P 7100 5750
-F 0 "TP16" H 7350 5750 60  0000 C CNN
-F 1 "TESTPAD" H 7150 5550 60  0001 C CNN
-F 2 "Anastasia:Test_Point_Round-SMD-Pad" H 7350 5750 60  0001 C CNN
-F 3 "" H 7350 5750 60  0000 C CNN
-	1    7100 5750
-	0    -1   -1   0
-$EndComp
-$Comp
-L TESTPAD TP13
-U 1 1 550CAB5D
-P 4800 3450
-F 0 "TP13" H 5050 3450 60  0000 C CNN
-F 1 "TESTPAD" H 4850 3250 60  0001 C CNN
-F 2 "Anastasia:Test_Point_Round-SMD-Pad" H 5050 3450 60  0001 C CNN
-F 3 "" H 5050 3450 60  0000 C CNN
-	1    4800 3450
-	1    0    0    -1
-$EndComp
-Wire Wire Line
-	4700 3450 4800 3450
-Connection ~ 7100 5750
+Wire Wire Line
+	2000 6450 2250 6450
+Wire Wire Line
+	2250 6450 2250 5750
+Connection ~ 2250 5750
+Wire Wire Line
+	2150 6650 2150 6000
+Connection ~ 2150 6000
+Connection ~ 2650 4800
+Connection ~ 2600 3950
 $EndSCHEMATC

Commit message: Refactoring
Parts:
- C13: value 0.1U -> 100N
Connections:
- wire segments 96 -> 119
Other:
- note added: "Battery Gauge\n"
- note removed: "A decoupling cap\n"
Changed lines of the file:
@@
 LIBS:memory
 LIBS:xilinx
-LIBS:special
 LIBS:microcontrollers
 LIBS:dsp
@@
 U 1 1 5504745A
 P 2250 1200
+AR Path="/5504745A" Ref="C1"  Part="1"
+AR Path="/55046F13/5504745A" Ref="C1"  Part="1"
 F 0 "C1" H 2300 1300 50  0000 L CNN
 F 1 "100N" H 2300 1100 50  0000 L CNN
@@
 U 1 1 5504747C
 P 2950 2350
+AR Path="/5504747C" Ref="C5"  Part="1"
+AR Path="/55046F13/5504747C" Ref="C5"  Part="1"
 F 0 "C5" H 3000 2450 50  0000 L CNN
 F 1 "10U" H 3000 2250 50  0000 L CNN
@@
 U 1 1 55047483
 P 3300 2350
+AR Path="/55047483" Ref="C6"  Part="1"
+AR Path="/55046F13/55047483" Ref="C6"  Part="1"
 F 0 "C6" H 3350 2450 50  0000 L CNN
 F 1 "10N" H 3350 2250 50  0000 L CNN
@@
 U 1 1 5504748A
 P 3550 2350
+AR Path="/5504748A" Ref="C7"  Part="1"
+AR Path="/55046F13/5504748A" Ref="C7"  Part="1"
 F 0 "C7" H 3600 2450 50  0000 L CNN
 F 1 "10N" H 3600 2250 50  0000 L CNN
@@
 U 1 1 55047497
 P 6250 1450
+AR Path="/55047497" Ref="C2"  Part="1"
+AR Path="/55046F13/55047497" Ref="C2"  Part="1"
 F 0 "C2" H 6300 1550 50  0000 L CNN
 F 1 "1U" H 6300 1350 50  0000 L CNN
@@
 U 1 1 550474B1
 P 6100 2550
+AR Path="/550474B1" Ref="C8"  Part="1"
+AR Path="/55046F13/550474B1" Ref="C8"  Part="1"
 F 0 "C8" H 6150 2650 50  0000 L CNN
 F 1 "100N" H 6150 2450 50  0000 L CNN
@@
 U 1 1 550474B8
 P 6350 2550
+AR Path="/550474B8" Ref="C9"  Part="1"
+AR Path="/55046F13/550474B8" Ref="C9"  Part="1"
 F 0 "C9" H 6400 2650 50  0000 L CNN
 F 1 "100N" H 6400 2450 50  0000 L CNN
@@
 U 1 1 550474BF
 P 6600 2550
+AR Path="/550474BF" Ref="C10"  Part="1"
+AR Path="/55046F13/550474BF" Ref="C10"  Part="1"
 F 0 "C10" H 6650 2650 50  0000 L CNN
 F 1 "100N" H 6650 2450 50  0000 L CNN
@@
 U 1 1 550474C6
 P 6950 2550
+AR Path="/550474C6" Ref="C11"  Part="1"
+AR Path="/55046F13/550474C6" Ref="C11"  Part="1"
 F 0 "C11" H 7000 2650 50  0000 L CNN
 F 1 "10U" H 7000 2450 50  0000 L CNN
@@
 	1    0    0    -1
 $EndComp
-Text Notes 6450 1500 0    60   ~ 0
-A decoupling cap\n
 Text Notes 6050 3050 0    60   ~ 0
 Power capacitors
@@
 U 1 1 550474F1
 P 1650 5000
+AR Path="/550474F1" Ref="C13"  Part="1"
+AR Path="/55046F13/550474F1" Ref="C13"  Part="1"
 F 0 "C13" H 1700 5100 50  0000 L CNN
-F 1 "0.1U" H 1700 4900 50  0000 L CNN
+F 1 "100N" H 1700 4900 50  0000 L CNN
 F 2 "Capacitors_SMD:C_0603" H 1688 4850 30  0001 C CNN
 F 3 "" H 1650 5000 60  0000 C CNN
@@
 U 1 1 550474FF
 P 4700 3800
+AR Path="/550474FF" Ref="C12"  Part="1"
+AR Path="/55046F13/550474FF" Ref="C12"  Part="1"
 F 0 "C12" H 4750 3900 50  0000 L CNN
 F 1 "2.2U" H 4750 3700 50  0000 L CNN
@@
 U 1 1 5504751C
 P 3400 1700
+AR Path="/5504751C" Ref="C3"  Part="1"
+AR Path="/55046F13/5504751C" Ref="C3"  Part="1"
 F 0 "C3" V 3450 1800 50  0000 L CNN
 F 1 "4.7U" V 3350 1450 50  0000 L CNN
@@
 U 1 1 55047523
 P 3400 1950
+AR Path="/55047523" Ref="C4"  Part="1"
+AR Path="/55046F13/55047523" Ref="C4"  Part="1"
 F 0 "C4" V 3450 2050 50  0000 L CNN
 F 1 "1U" V 3450 1700 50  0000 L CNN
@@
 U 1 1 550479A6
 P 7250 6000
+AR Path="/550479A6" Ref="C14"  Part="1"
+AR Path="/55046F13/550479A6" Ref="C14"  Part="1"
 F 0 "C14" H 7300 6100 50  0000 L CNN
 F 1 "4.7U" H 7300 5900 50  0000 L CNN
@@
 U 1 1 55085D1A
 P 6500 6050
+AR Path="/55085D1A" Ref="C15"  Part="1"
+AR Path="/55046F13/55085D1A" Ref="C15"  Part="1"
 F 0 "C15" H 6550 6150 50  0000 L CNN
 F 1 "0.47U" H 6550 5950 50  0000 L CNN
@@
 	0    1    1    0
 $EndComp
+Text HLabel 4900 6200 0    60   Input ~ 0
+GPOUT
+Text HLabel 4900 5600 0    60   Input ~ 0
+GAUGE_SCL
+Text HLabel 4900 5700 0    60   Input ~ 0
+GAUGE_SDA
+$Comp
+L IP4220CZ6 U4
+U 1 1 55094F19
+P 1150 6350
+F 0 "U4" H 1200 6400 60  0000 C CNN
+F 1 "IP4220CZ6" H 1550 5900 60  0000 C CNN
+F 2 "Anastasia:SOT457" H 1150 6350 60  0001 C CNN
+F 3 "" H 1150 6350 60  0000 C CNN
+	1    1150 6350
+	1    0    0    -1
+$EndComp
+NoConn ~ 950  6450
+NoConn ~ 950  6650
+Text GLabel 2250 6550 2    60   Input ~ 0
+USB_VBUS
+$Comp
+L GND #PWR060
+U 1 1 550950F7
+P 650 6550
+F 0 "#PWR060" H 650 6300 60  0001 C CNN
+F 1 "GND" H 650 6400 60  0000 C CNN
+F 2 "" H 650 6550 60  0000 C CNN
+F 3 "" H 650 6550 60  0000 C CNN
+	1    650  6550
+	1    0    0    -1
+$EndComp
+Text Notes 1150 6950 0    60   ~ 0
+ESD Protection\n
+Text Notes 4000 4350 0    60   ~ 0
+Battery Charge Current Set Resistor
 Wire Wire Line
 	3800 3850 3700 3850
 Wire Wire Line
-	1700 3700 1700 3600
-Wire Wire Line
-	1700 4250 1700 4200
-Wire Wire Line
-	2600 4250 1700 4250
+	1700 3600 1700 3800
+Wire Wire Line
+	1700 4100 1700 4250
+Wire Wire Line
+	1700 4250 2600 4250
 Wire Wire Line
 	2500 4150 2600 4150
@@
 	3700 3950 3700 4050
 Wire Wire Line
-	3650 6000 3350 6000
-Wire Wire Line
-	3650 5750 3350 5750
+	3250 6000 3650 6000
+Wire Wire Line
+	3250 5750 3650 5750
 Connection ~ 2850 6000
 Connection ~ 2850 5750
 Wire Wire Line
-	1900 6000 2850 6000
-Wire Wire Line
-	2050 5750 2850 5750
+	1900 6000 2950 6000
+Wire Wire Line
+	2050 5750 2950 5750
 Wire Wire Line
 	2650 5000 2050 5000
@@
 	2050 1950 2050 2150
 Wire Wire Line
-	2050 2150 2250 2150
-Wire Wire Line
-	2750 2150 3750 2150
+	2050 2150 2350 2150
+Wire Wire Line
+	2650 2150 3750 2150
 Wire Wire Line
 	2750 2650 2750 2550
@@
 	5950 2350 6950 2350
 Wire Wire Line
-	6950 2350 6950 2250
+	6950 2250 6950 2400
 Wire Wire Line
 	5950 2750 6950 2750
@@
 	1550 4800 2650 4800
 Wire Wire Line
-	3650 5400 1650 5400
+	1650 5400 3650 5400
 Connection ~ 2100 4800
 Connection ~ 2250 5400
@@
 	4500 3650 4700 3600
 Wire Wire Line
-	4700 4000 4700 4100
-Wire Wire Line
-	4700 3600 4700 3450
-Wire Wire Line
-	4350 4150 4600 4150
+	4700 3950 4700 4100
+Wire Wire Line
+	4700 3450 4700 3650
+Wire Wire Line
+	4250 4150 4600 4150
 Wire Wire Line
 	4600 4150 4600 4000
@@
 	4600 4000 4700 4000
 Wire Wire Line
-	3850 4150 3700 4150
+	3700 4150 3950 4150
 Connection ~ 1650 4800
 Wire Wire Line
@@
 	3750 1550 3750 1750
 Wire Wire Line
-	3750 1700 3600 1700
+	3550 1700 3750 1700
 Connection ~ 3750 1700
 Wire Wire Line
-	3750 1850 3750 1950
-Wire Wire Line
-	3750 1950 3600 1950
-Wire Wire Line
-	2950 1700 3200 1700
+	3750 1950 3750 1850
+Wire Wire Line
+	3550 1950 3750 1950
+Wire Wire Line
+	2950 1700 3250 1700
 Wire Wire Line
 	2950 1850 2950 1700
@@
 	3200 1850 2950 1850
 Wire Wire Line
-	1650 5400 1650 5200
+	1650 5150 1650 5400
 Wire Wire Line
 	2650 5400 2650 5200
 Wire Wire Line
-	3650 4800 3650 5400
+	3650 5400 3650 4800
 Connection ~ 3650 4900
 Connection ~ 3650 5100
@@
 	5000 5900 4950 5900
 Wire Wire Line
-	4450 5850 4400 5850
+	4400 5850 4550 5850
 Wire Wire Line
 	4950 5900 4950 5850
-Text HLabel 4900 6200 0    60   Input ~ 0
-GPOUT
-Text HLabel 4900 5600 0    60   Input ~ 0
-GAUGE_SCL
-Text HLabel 4900 5700 0    60   Input ~ 0
-GAUGE_SDA
 Wire Wire Line
 	4900 5600 5000 5600
@@
 Wire Wire Line
 	4900 6000 5000 6000
-$Comp
-L IP4220CZ6 U4
-U 1 1 55094F19
-P 1150 6350
-F 0 "U4" H 1200 6400 60  0000 C CNN
-F 1 "IP4220CZ6" H 1550 5900 60  0000 C CNN
-F 2 "Anastasia:SOT457" H 1150 6350 60  0001 C CNN
-F 3 "" H 1150 6350 60  0000 C CNN
-	1    1150 6350
-	1    0    0    -1
-$EndComp
-NoConn ~ 950  6450
-NoConn ~ 950  6650
-Text GLabel 2250 6550 2    60   Input ~ 0
-USB_VBUS
 Wire Wire Line
 	2250 6550 2000 6550
-$Comp
-L GND #PWR060
-U 1 1 550950F7
-P 650 6550
-F 0 "#PWR060" H 650 6300 60  0001 C CNN
-F 1 "GND" H 650 6400 60  0000 C CNN
-F 2 "" H 650 6550 60  0000 C CNN
-F 3 "" H 650 6550 60  0000 C CNN
-	1    650  6550
-	1    0    0    -1
-$EndComp
 Wire Wire Line
 	950  6550 650  6550
@@
 Wire Wire Line
 	2000 6650 2150 6650
-Text Notes 1150 6950 0    60   ~ 0
-ESD Protection\n
-Text Notes 4000 4350 0    60   ~ 0
-Battery Charge Current Set Resistor
 Connection ~ 4400 5850
 Wire Wire Line
 	7400 5800 7250 5800
 Wire Wire Line
-	7250 5800 7250 5750
+	7250 5750 7250 5850
 Wire Wire Line
 	4450 5150 6100 5150
@@
 Connection ~ 2650 4800
 Connection ~ 2600 3950
+Wire Wire Line
+	2250 1400 2250 1350
+Wire Wire Line
+	2250 1050 2250 1000
+Wire Wire Line
+	3200 1950 3250 1950
+Wire Wire Line
+	2950 2550 2950 2500
+Wire Wire Line
+	2950 2200 2950 2150
+Wire Wire Line
+	3300 2200 3300 2150
+Wire Wire Line
+	3550 2150 3550 2200
+Wire Wire Line
+	3550 2550 3550 2500
+Wire Wire Line
+	3300 2500 3300 2550
+Wire Wire Line
+	6250 1600 6250 1650
+Wire Wire Line
+	6250 1250 6250 1300
+Wire Wire Line
+	6100 2400 6100 2350
+Wire Wire Line
+	6350 2400 6350 2350
+Wire Wire Line
+	6600 2400 6600 2350
+Wire Wire Line
+	6950 2750 6950 2700
+Wire Wire Line
+	6600 2750 6600 2700
+Wire Wire Line
+	6350 2750 6350 2700
+Wire Wire Line
+	6100 2750 6100 2700
+Wire Wire Line
+	7250 6200 7250 6150
+Wire Wire Line
+	6500 6250 6500 6200
+Wire Wire Line
+	6500 5850 6500 5900
+Wire Wire Line
+	4950 5850 4850 5850
+Wire Wire Line
+	1650 4850 1650 4800
+Connection ~ 4700 4000
+Connection ~ 4700 3600
+Text Notes 5250 6500 0    60   ~ 0
+Battery Gauge\n
 $EndSCHEMATC
