File: KiCad project/Sheet2.sch (KiCad schematic (older format))
At the start: 7 parts, among them U1 EFM32GG332, X1 SMD_32.768kHz_CRYSTAL_OSC, X2 SMD_48MHZ_CRYSTAL_OSC

Commit message: Bluetooth schematics
nRF8001 schematics, various additions and modification, test points
added
Changed lines of the file:
@@
 $Descr A4 11693 8268
 encoding utf-8
-Sheet 3 4
+Sheet 3 6
 Title "uC part A"
 Date "14 March 2015"
@@
 	4700 3200 4700 3050
 $Comp
-L GND #PWR13
+L GND #PWR014
 U 1 1 5504D536
 P 4900 2500
-F 0 "#PWR13" H 4900 2250 60  0001 C CNN
+F 0 "#PWR014" H 4900 2250 60  0001 C CNN
 F 1 "GND" H 4900 2350 60  0000 C CNN
 F 2 "" H 4900 2500 60  0000 C CNN
@@
 $EndComp
 Wire Wire Line
-	4700 2500 4900 2500
-Wire Wire Line
-	4900 2500 5100 2500
+	4700 2500 5100 2500
 Wire Wire Line
 	5100 2500 5100 2650
@@
 $EndComp
 Wire Wire Line
-	5350 1950 5550 1950
-Wire Wire Line
-	5550 1950 5750 1950
+	5350 1950 5750 1950
 Wire Wire Line
 	4900 2500 4900 1800
@@
 Connection ~ 5550 1950
 Wire Wire Line
-	5350 2350 5350 2500
-Wire Wire Line
-	5350 2500 5350 2950
+	5350 2350 5350 2950
 Wire Wire Line
 	5750 2500 5750 2350
@@
 Connection ~ 5350 2500
 $Comp
-L GND #PWR15
+L GND #PWR015
 U 1 1 5504D88A
 P 4900 3300
-F 0 "#PWR15" H 4900 3050 60  0001 C CNN
+F 0 "#PWR015" H 4900 3050 60  0001 C CNN
 F 1 "GND" H 4900 3150 60  0000 C CNN
 F 2 "" H 4900 3300 60  0000 C CNN
@@
 $EndComp
 $Comp
-L GND #PWR14
+L GND #PWR016
 U 1 1 5504D89E
 P 5550 2600
-F 0 "#PWR14" H 5550 2350 60  0001 C CNN
+F 0 "#PWR016" H 5550 2350 60  0001 C CNN
 F 1 "GND" H 5550 2450 60  0000 C CNN
 F 2 "" H 5550 2600 60  0000 C CNN
