File: KiCad project/$Anastasia.sch (KiCad schematic (older format))
At the start: 11 parts

Commit message: IC packages, bugfixes
drawings for IC packages, associations, schematic fixes
Parts:
- renumbered TP6 to TP1, TP15 to TP10, TP16 to TP11, TP7 to TP2, TP8 to TP3, TP9 to TP4, TP10 to TP5, TP11 to TP6, TP12 to TP7, TP13 to TP8, TP14 to TP9
Changed lines of the file:
@@
 Connection ~ 4400 2950
 $Comp
-L TESTPAD TP6
+L TESTPAD TP1
 U 1 1 550D1F0B
 P 2200 1000
-F 0 "TP6" H 2450 1000 60  0000 C CNN
+F 0 "TP1" H 2450 1000 60  0000 C CNN
 F 1 "TESTPAD" H 2250 800 60  0001 C CNN
 F 2 "" H 2450 1000 60  0000 C CNN
@@
 $EndComp
 $Comp
-L TESTPAD TP7
+L TESTPAD TP2
 U 1 1 550D1F40
 P 2350 1000
-F 0 "TP7" H 2600 1000 60  0000 C CNN
+F 0 "TP2" H 2600 1000 60  0000 C CNN
 F 1 "TESTPAD" H 2400 800 60  0001 C CNN
 F 2 "" H 2600 1000 60  0000 C CNN
@@
 $EndComp
 $Comp
-L TESTPAD TP8
+L TESTPAD TP3
 U 1 1 550D1F5F
 P 2500 1000
-F 0 "TP8" H 2750 1000 60  0000 C CNN
+F 0 "TP3" H 2750 1000 60  0000 C CNN
 F 1 "TESTPAD" H 2550 800 60  0001 C CNN
 F 2 "" H 2750 1000 60  0000 C CNN
@@
 $EndComp
 $Comp
-L TESTPAD TP9
+L TESTPAD TP4
 U 1 1 550D1F7E
 P 2650 1000
-F 0 "TP9" H 2900 1000 60  0000 C CNN
+F 0 "TP4" H 2900 1000 60  0000 C CNN
 F 1 "TESTPAD" H 2700 800 60  0001 C CNN
 F 2 "" H 2900 1000 60  0000 C CNN
@@
 Connection ~ 2650 1550
 $Comp
-L TESTPAD TP10
+L TESTPAD TP5
 U 1 1 550D353F
 P 4300 1000
-F 0 "TP10" H 4550 1000 60  0000 C CNN
+F 0 "TP5" H 4550 1000 60  0000 C CNN
 F 1 "TESTPAD" H 4350 800 60  0001 C CNN
 F 2 "" H 4550 1000 60  0000 C CNN
@@
 $EndComp
 $Comp
-L TESTPAD TP11
+L TESTPAD TP6
 U 1 1 550D3564
 P 4500 1000
-F 0 "TP11" H 4750 1000 60  0000 C CNN
+F 0 "TP6" H 4750 1000 60  0000 C CNN
 F 1 "TESTPAD" H 4550 800 60  0001 C CNN
 F 2 "" H 4750 1000 60  0000 C CNN
@@
 $EndComp
 $Comp
-L TESTPAD TP15
+L TESTPAD TP10
 U 1 1 550D3583
 P 4300 3100
-F 0 "TP15" H 4550 3100 60  0000 C CNN
+F 0 "TP10" H 4550 3100 60  0000 C CNN
 F 1 "TESTPAD" H 4350 2900 60  0001 C CNN
 F 2 "" H 4550 3100 60  0000 C CNN
@@
 $EndComp
 $Comp
-L TESTPAD TP16
+L TESTPAD TP11
 U 1 1 550D359E
 P 4400 3100
-F 0 "TP16" H 4650 3100 60  0000 C CNN
+F 0 "TP11" H 4650 3100 60  0000 C CNN
 F 1 "TESTPAD" H 4450 2900 60  0001 C CNN
 F 2 "" H 4650 3100 60  0000 C CNN
@@
 Connection ~ 4500 1350
 $Comp
-L TESTPAD TP13
+L TESTPAD TP8
 U 1 1 550D3905
 P 7750 2900
-F 0 "TP13" H 8000 2900 60  0000 C CNN
+F 0 "TP8" H 8000 2900 60  0000 C CNN
 F 1 "TESTPAD" H 7800 2700 60  0001 C CNN
 F 2 "" H 8000 2900 60  0000 C CNN
@@
 $EndComp
 $Comp
-L TESTPAD TP14
+L TESTPAD TP9
 U 1 1 550D3920
 P 7950 2900
-F 0 "TP14" H 8200 2900 60  0000 C CNN
+F 0 "TP9" H 8200 2900 60  0000 C CNN
 F 1 "TESTPAD" H 8000 2700 60  0001 C CNN
 F 2 "" H 8200 2900 60  0000 C CNN
@@
 Connection ~ 7950 2600
 $Comp
-L TESTPAD TP12
+L TESTPAD TP7
 U 1 1 550D3AEA
 P 7600 2350
-F 0 "TP12" H 7850 2350 60  0000 C CNN
+F 0 "TP7" H 7850 2350 60  0000 C CNN
 F 1 "TESTPAD" H 7650 2150 60  0001 C CNN
 F 2 "" H 7850 2350 60  0000 C CNN
