File: KiCad project/_autosave-Anastasia.kicad_pcb (KiCad board)
At the start: 4 copper layers, 32 x 33 mm, 95 parts, among them CON1 USB-MICRO-B, P1 LS013B4DN04, U1 EFM32GG332, U2 BQ25011, U3 BQ27421-G1, U4 IP4220CZ6, U5 MPU-9150, U6 AT24CM01, U7 AFE4403, U8 nRF8001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

Commit message: New packages, PCB
Parts:
- added TP19: TESTPAD, Measurement_Points:Measurement_Point_Round-SMD-Pad_Small, F.Cu at (84.2, 55.8)
- added TP20: TESTPAD, Measurement_Points:Measurement_Point_Round-SMD-Pad_Small, F.Cu at (90.8, 65.2)
- added TP21: TESTPAD, Measurement_Points:Measurement_Point_Round-SMD-Pad_Small, F.Cu at (94.0, 57.8)
- added TP22: TESTPAD, Measurement_Points:Measurement_Point_Round-SMD-Pad_Small, F.Cu at (82.8, 69.0)
- added TP23: TESTPAD, Measurement_Points:Measurement_Point_Round-SMD-Pad_Small, F.Cu at (82.0, 59.5)
- added TP24: TESTPAD, Measurement_Points:Measurement_Point_Round-SMD-Pad_Small, F.Cu at (88.2, 58.5)
- added TP25: TESTPAD, Measurement_Points:Measurement_Point_Round-SMD-Pad_Small, F.Cu at (75.5, 76.2)
- added TP26: TESTPAD, Measurement_Points:Measurement_Point_Round-SMD-Pad_Small, F.Cu at (82.5, 79.0)
- added TP27: TESTPAD, Measurement_Points:Measurement_Point_Round-SMD-Pad_Small, F.Cu at (104.2, 80.2)
- added TP28: TESTPAD, Measurement_Points:Measurement_Point_Round-SMD-Pad_Small, F.Cu at (86.0, 63.1)
- U7: moved to B.Cu
- moved U7 63.9 mm to (79.2, 24.0)
- moved R3 53.6 mm to (134.0, 87.0)
- moved R2 50.2 mm to (123.0, 97.0)
- moved R6 49.2 mm to (130.0, 85.0)
- moved L1 48.5 mm to (127.0, 89.0)
- moved R4 48.1 mm to (131.0, 80.0)
- moved R8 44.8 mm to (114.0, 98.0)
- moved R5 44.8 mm to (125.0, 85.0)
- moved L2 43.4 mm to (128.0, 74.0)
- moved C43 43.1 mm to (126.0, 79.0)
- moved L5 41.3 mm to (127.0, 68.0)
- moved C44 40.8 mm to (119.0, 87.0)
- moved R1 38.9 mm to (120.0, 82.0)
- moved C45 38.9 mm to (114.0, 90.0)
- moved L3 38.6 mm to (123.0, 74.0)
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