File: KiCad project/Sheet5.sch (KiCad schematic (older format))
At the start: 22 parts, among them U4 nRF8001, X3 CRYSTAL_SMD_16MHZ

Commit message: IC packages, bugfixes
drawings for IC packages, associations, schematic fixes
Parts:
- C36: footprint (none) -> Resistors_SMD:R_0603_HandSoldering
- U4: footprint (none) -> Anastasia:QFN32
Changed lines of the file:
@@
 $Descr A4 11693 8268
 encoding utf-8
-Sheet 6 7
+Sheet 10 10
 Title "nRF8001"
 Date "15 March 2015"
@@
 F 0 "U4" H 5350 1250 60  0000 C CNN
 F 1 "nRF8001" H 5900 -950 60  0000 C CNN
-F 2 "" H 5300 1200 60  0000 C CNN
+F 2 "Anastasia:QFN32" H 5300 1200 60  0001 C CNN
 F 3 "" H 5300 1200 60  0000 C CNN
 	1    5300 1200
@@
 F 0 "C25" H 4100 1600 50  0000 L CNN
 F 1 "4.7U" H 4100 1400 50  0000 L CNN
-F 2 "" H 4088 1350 30  0000 C CNN
+F 2 "" H 4088 1350 30  0001 C CNN
 F 3 "" H 4050 1500 60  0000 C CNN
 	1    4050 1500
@@
 $EndComp
 $Comp
-L +3V3 #PWR27
+L +3V3 #PWR048
 U 1 1 550557EE
 P 4050 1150
-F 0 "#PWR27" H 4050 1000 60  0001 C CNN
+F 0 "#PWR048" H 4050 1000 60  0001 C CNN
 F 1 "+3V3" H 4050 1290 60  0000 C CNN
 F 2 "" H 4050 1150 60  0000 C CNN
@@
 $EndComp
 $Comp
-L GND #PWR31
+L GND #PWR049
 U 1 1 55055802
 P 4050 1850
-F 0 "#PWR31" H 4050 1600 60  0001 C CNN
+F 0 "#PWR049" H 4050 1600 60  0001 C CNN
 F 1 "GND" H 4050 1700 60  0000 C CNN
 F 2 "" H 4050 1850 60  0000 C CNN
@@
 F 0 "C30" H 4250 3050 50  0000 L CNN
 F 1 "100N" H 4250 2850 50  0000 L CNN
-F 2 "" H 4238 2800 30  0000 C CNN
+F 2 "" H 4238 2800 30  0001 C CNN
 F 3 "" H 4200 2950 60  0000 C CNN
 	1    4200 2950
@@
 F 0 "C32" H 4600 3150 50  0000 L CNN
 F 1 "33N" H 4600 2950 50  0000 L CNN
-F 2 "" H 4588 2900 30  0000 C CNN
+F 2 "" H 4588 2900 30  0001 C CNN
 F 3 "" H 4550 3050 60  0000 C CNN
 	1    4550 3050
@@
 $EndComp
 $Comp
-L GND #PWR38
+L GND #PWR050
 U 1 1 5505586E
 P 4400 3400
-F 0 "#PWR38" H 4400 3150 60  0001 C CNN
+F 0 "#PWR050" H 4400 3150 60  0001 C CNN
 F 1 "GND" H 4400 3250 60  0000 C CNN
 F 2 "" H 4400 3400 60  0000 C CNN
@@
 F 0 "C26" H 4450 1850 50  0000 L CNN
 F 1 "100N" H 4450 1650 50  0000 L CNN
-F 2 "" H 4438 1600 30  0000 C CNN
+F 2 "" H 4438 1600 30  0001 C CNN
 F 3 "" H 4400 1750 60  0000 C CNN
 	1    4400 1750
@@
 $EndComp
 $Comp
-L GND #PWR32
+L GND #PWR051
 U 1 1 5505597E
 P 4400 2050
-F 0 "#PWR32" H 4400 1800 60  0001 C CNN
+F 0 "#PWR051" H 4400 1800 60  0001 C CNN
 F 1 "GND" H 4400 1900 60  0000 C CNN
 F 2 "" H 4400 2050 60  0000 C CNN
@@
 F 0 "C27" H 4850 1950 50  0000 L CNN
 F 1 "1N" H 4850 1750 50  0000 L CNN
-F 2 "" H 4838 1700 30  0000 C CNN
+F 2 "" H 4838 1700 30  0001 C CNN
 F 3 "" H 4800 1850 60  0000 C CNN
 	1    4800 1850
@@
 $EndComp
 $Comp
-L GND #PWR33
+L GND #PWR052
 U 1 1 550559EB
 P 4800 2150
-F 0 "#PWR33" H 4800 1900 60  0001 C CNN
+F 0 "#PWR052" H 4800 1900 60  0001 C CNN
 F 1 "GND" H 4800 2000 60  0000 C CNN
 F 2 "" H 4800 2150 60  0000 C CNN
@@
 	5150 1650 4800 1650
 $Comp
-L +3V3 #PWR30
+L +3V3 #PWR053
 U 1 1 55055A52
 P 4800 1600
-F 0 "#PWR30" H 4800 1450 60  0001 C CNN
+F 0 "#PWR053" H 4800 1450 60  0001 C CNN
 F 1 "+3V3" H 4800 1740 60  0000 C CNN
 F 2 "" H 4800 1600 60  0000 C CNN
@@
 	4800 1650 4800 1600
 $Comp
-L +3V3 #PWR29
+L +3V3 #PWR054
 U 1 1 55055A97
 P 4400 1500
-F 0 "#PWR29" H 4400 1350 60  0001 C CNN
+F 0 "#PWR054" H 4400 1350 60  0001 C CNN
 F 1 "+3V3" H 4400 1640 60  0000 C CNN
 F 2 "" H 4400 1500 60  0000 C CNN
@@
 	4550 1550 4400 1550
 $Comp
-L GND #PWR34
+L GND #PWR055
 U 1 1 55055AEC
 P 4950 2250
-F 0 "#PWR34" H 4950 2000 60  0001 C CNN
+F 0 "#PWR055" H 4950 2000 60  0001 C CNN
 F 1 "GND" H 4950 2100 60  0000 C CNN
 F 2 "" H 4950 2250 60  0000 C CNN
@@
 	5150 2250 4950 2250
 Wire Wire Line
-	5150 1950 5150 2450
+	5150 1850 5150 2450
 Connection ~ 5150 2350
 Connection ~ 5150 2250
@@
 F 0 "R5" V 6730 1450 50  0000 C CNN
 F 1 "22K" V 6657 1451 50  0000 C CNN
-F 2 "" V 6580 1450 30  0000 C CNN
+F 2 "" V 6580 1450 30  0001 C CNN
 F 3 "" H 6650 1450 30  0000 C CNN
 	1    6650 1450
@@
 $EndComp
 $Comp
-L GND #PWR28
+L GND #PWR056
 U 1 1 55068568
 P 7100 1450
-F 0 "#PWR28" H 7100 1200 60  0001 C CNN
+F 0 "#PWR056" H 7100 1200 60  0001 C CNN
 F 1 "GND" H 7100 1300 60  0000 C CNN
 F 2 "" H 7100 1450 60  0000 C CNN
@@
 Wire Wire Line
 	6250 1450 6400 1450
-Wire Wire Line
-	6900 1450 7100 1450
 $Comp
 L INDUCTOR L5
@@
 F 0 "L5" V 7350 3100 50  0000 C CNN
 F 1 "8.2NH" V 7500 3100 50  0000 C CNN
-F 2 "" H 7400 3100 60  0000 C CNN
+F 2 "" H 7400 3100 60  0001 C CNN
 F 3 "" H 7400 3100 60  0000 C CNN
 	1    7400 3100
@@
 F 0 "L4" V 7850 2800 50  0000 C CNN
 F 1 "5.6NH" V 8000 2800 50  0000 C CNN
-F 2 "" H 7900 2800 60  0000 C CNN
+F 2 "" H 7900 2800 60  0001 C CNN
 F 3 "" H 7900 2800 60  0000 C CNN
 	1    7900 2800
@@
 F 0 "L6" V 7850 3400 50  0000 C CNN
 F 1 "3.9NH" V 8000 3400 50  0000 C CNN
-F 2 "" H 7900 3400 60  0000 C CNN
+F 2 "" H 7900 3400 60  0001 C CNN
 F 3 "" H 7900 3400 60  0000 C CNN
 	1    7900 3400
@@
 F 0 "C35" H 9300 4250 50  0000 L CNN
 F 1 "2.2N" H 9300 4050 50  0000 L CNN
-F 2 "" H 9288 4000 30  0000 C CNN
+F 2 "" H 9288 4000 30  0001 C CNN
 F 3 "" H 9250 4150 60  0000 C CNN
 	1    9250 4150
@@
 F 0 "C36" H 9750 4250 50  0000 L CNN
 F 1 "N/C" H 9750 4050 50  0000 L CNN
-F 2 "" H 9738 4000 30  0000 C CNN
+F 2 "Resistors_SMD:R_0603_HandSoldering" H 9738 4000 30  0001 C CNN
 F 3 "" H 9700 4150 60  0000 C CNN
 	1    9700 4150
@@
 	9700 4350 9250 4350
 $Comp
-L GND #PWR40
+L GND #PWR057
 U 1 1 55068D17
 P 9500 4350
-F 0 "#PWR40" H 9500 4100 60  0001 C CNN
+F 0 "#PWR057" H 9500 4100 60  0001 C CNN
 F 1 "GND" H 9500 4200 60  0000 C CNN
 F 2 "" H 9500 4350 60  0000 C CNN
@@
 F 0 "C33" H 8550 3500 50  0000 L CNN
 F 1 "1.8N" H 8550 3300 50  0000 L CNN
-F 2 "" H 8538 3250 30  0000 C CNN
+F 2 "" H 8538 3250 30  0001 C CNN
 F 3 "" H 8500 3400 60  0000 C CNN
 	1    8500 3400
@@
 F 0 "C34" H 8850 3700 50  0000 L CNN
 F 1 "1.2N" H 8850 3500 50  0000 L CNN
-F 2 "" H 8838 3450 30  0000 C CNN
+F 2 "" H 8838 3450 30  0001 C CNN
 F 3 "" H 8800 3600 60  0000 C CNN
 	1    8800 3600
@@
 $EndComp
 $Comp
-L GND #PWR39
+L GND #PWR058
 U 1 1 55068D89
 P 9000 3750
-F 0 "#PWR39" H 9000 3500 60  0001 C CNN
+F 0 "#PWR058" H 9000 3500 60  0001 C CNN
 F 1 "GND" H 9000 3600 60  0000 C CNN
 F 2 "" H 9000 3750 60  0000 C CNN
@@
 F 0 "L3" V 3500 2600 50  0000 C CNN
 F 1 "10UH" V 3650 2600 50  0000 C CNN
-F 2 "" H 3550 2600 60  0000 C CNN
+F 2 "" H 3550 2600 60  0001 C CNN
 F 3 "" H 3550 2600 60  0000 C CNN
 	1    3550 2600
@@
 F 0 "L2" V 2750 2600 50  0000 C CNN
 F 1 "15NH" V 2900 2600 50  0000 C CNN
-F 2 "" H 2800 2600 60  0000 C CNN
+F 2 "" H 2800 2600 60  0001 C CNN
 F 3 "" H 2800 2600 60  0000 C CNN
 	1    2800 2600
@@
 F 0 "C31" H 2550 3150 50  0000 L CNN
 F 1 "1U" H 2550 2950 50  0000 L CNN
-F 2 "" H 2538 2900 30  0000 C CNN
+F 2 "" H 2538 2900 30  0001 C CNN
 F 3 "" H 2500 3050 60  0000 C CNN
 	1    2500 3050
@@
 Connection ~ 2500 2600
 $Comp
-L +3V3 #PWR36
+L +3V3 #PWR059
 U 1 1 55069C09
 P 2500 2450
-F 0 "#PWR36" H 2500 2300 60  0001 C CNN
+F 0 "#PWR059" H 2500 2300 60  0001 C CNN
 F 1 "+3V3" H 2500 2590 60  0000 C CNN
 F 2 "" H 2500 2450 60  0000 C CNN
@@
 $EndComp
 $Comp
-L GND #PWR37
+L GND #PWR060
 U 1 1 55069C1D
 P 2500 3350
-F 0 "#PWR37" H 2500 3100 60  0001 C CNN
+F 0 "#PWR060" H 2500 3100 60  0001 C CNN
 F 1 "GND" H 2500 3200 60  0000 C CNN
 F 2 "" H 2500 3350 60  0000 C CNN
@@
 F 0 "X3" H 8100 1740 50  0000 C CNN
 F 1 "CRYSTAL_SMD_16MHZ" H 8130 1540 50  0000 L CNN
-F 2 "" H 8100 1650 60  0000 C CNN
+F 2 "" H 8100 1650 60  0001 C CNN
 F 3 "" H 8100 1650 60  0000 C CNN
 	1    8100 1650
@@
 F 0 "C28" H 7950 2150 50  0000 L CNN
 F 1 "12P" H 7950 1950 50  0000 L CNN
-F 2 "" H 7938 1900 30  0000 C CNN
+F 2 "" H 7938 1900 30  0001 C CNN
 F 3 "" H 7900 2050 60  0000 C CNN
 	1    7900 2050
@@
 F 0 "C29" H 8350 2150 50  0000 L CNN
 F 1 "12P" H 8350 1950 50  0000 L CNN
-F 2 "" H 8338 1900 30  0000 C CNN
+F 2 "" H 8338 1900 30  0001 C CNN
 F 3 "" H 8300 2050 60  0000 C CNN
 	1    8300 2050
@@
 $EndComp
 $Comp
-L GND #PWR35
+L GND #PWR061
 U 1 1 5506A4BA
 P 8100 2300
-F 0 "#PWR35" H 8100 2050 60  0001 C CNN
+F 0 "#PWR061" H 8100 2050 60  0001 C CNN
 F 1 "GND" H 8100 2150 60  0000 C CNN
 F 2 "" H 8100 2300 60  0000 C CNN
@@
 F 0 "TP1" H 6600 2800 60  0000 C CNN
 F 1 "TESTPAD" H 6400 2600 60  0001 C CNN
-F 2 "" H 6600 2800 60  0000 C CNN
+F 2 "" H 6600 2800 60  0001 C CNN
 F 3 "" H 6600 2800 60  0000 C CNN
 	1    6350 2800
@@
 F 0 "TP2" H 6600 2900 60  0000 C CNN
 F 1 "TESTPAD" H 6400 2700 60  0001 C CNN
-F 2 "" H 6600 2900 60  0000 C CNN
+F 2 "" H 6600 2900 60  0001 C CNN
 F 3 "" H 6600 2900 60  0000 C CNN
 	1    6350 2900
@@
 Wire Wire Line
 	6250 2650 6450 2650
+Connection ~ 5150 1950
+Wire Wire Line
+	6900 1450 7100 1450
 $EndSCHEMATC

Commit message: New packages, PCB
Parts:
- C36: renamed from C25; footprint (none) -> Capacitors_SMD:C_0603
- C37: renamed from C26; footprint (none) -> Capacitors_SMD:C_0603
- C38: renamed from C27; footprint (none) -> Capacitors_SMD:C_0603
- C39: renamed from C28; value 12P -> 10P; footprint (none) -> Capacitors_SMD:C_0603
- C40: renamed from C29; value 12P -> 10P; footprint (none) -> Capacitors_SMD:C_0603
- C41: renamed from C30; footprint (none) -> Capacitors_SMD:C_0603
- C42: renamed from C31; footprint (none) -> Capacitors_SMD:C_0603
- C43: renamed from C32; footprint (none) -> Capacitors_SMD:C_0603
- C44: renamed from C33; footprint (none) -> Capacitors_SMD:C_0603
- C45: renamed from C34; footprint (none) -> Capacitors_SMD:C_0603
- C46: renamed from C35; footprint (none) -> Capacitors_SMD:C_0603
- L2, L3, L4, L5, L6: footprint (none) -> Resistors_SMD:R_0603
- R8: renamed from R5; footprint (none) -> Resistors_SMD:R_0603
- TP17: renamed from TP1; footprint (none) -> Measurement_Points:Measurement_Point_Round-SMD-Pad_Small
- TP18: renamed from TP2; footprint (none) -> Measurement_Points:Measurement_Point_Round-SMD-Pad_Small
- X4: renamed from X3; footprint (none) -> Anastasia:2x1.6CRYSTAL
- renumbered C36 to C47, U4 to U8
Connections:
- wire segments 61 -> 62

Commit message: Schematics, PCB design
New schematics for the pulse oximeter, PCB layout design
Changed lines of the file:
@@
 $EndComp
 $Comp
-L +3V3 #PWR047
+L +3V3 #PWR045
 U 1 1 550557EE
 P 4050 1150
-F 0 "#PWR047" H 4050 1000 60  0001 C CNN
+F 0 "#PWR045" H 4050 1000 60  0001 C CNN
 F 1 "+3V3" H 4050 1290 60  0000 C CNN
 F 2 "" H 4050 1150 60  0000 C CNN
@@
 $EndComp
 $Comp
-L GND #PWR048
+L GND #PWR046
 U 1 1 55055802
 P 4050 1850
-F 0 "#PWR048" H 4050 1600 60  0001 C CNN
+F 0 "#PWR046" H 4050 1600 60  0001 C CNN
 F 1 "GND" H 4050 1700 60  0000 C CNN
 F 2 "" H 4050 1850 60  0000 C CNN
@@
 $EndComp
 $Comp
-L GND #PWR049
+L GND #PWR047
 U 1 1 5505586E
 P 4400 3400
-F 0 "#PWR049" H 4400 3150 60  0001 C CNN
+F 0 "#PWR047" H 4400 3150 60  0001 C CNN
 F 1 "GND" H 4400 3250 60  0000 C CNN
 F 2 "" H 4400 3400 60  0000 C CNN
@@
 $EndComp
 $Comp
-L GND #PWR050
+L GND #PWR048
 U 1 1 5505597E
 P 4400 2050
-F 0 "#PWR050" H 4400 1800 60  0001 C CNN
+F 0 "#PWR048" H 4400 1800 60  0001 C CNN
 F 1 "GND" H 4400 1900 60  0000 C CNN
 F 2 "" H 4400 2050 60  0000 C CNN
@@
 $EndComp
 $Comp
-L GND #PWR051
+L GND #PWR049
 U 1 1 550559EB
 P 4800 2150
-F 0 "#PWR051" H 4800 1900 60  0001 C CNN
+F 0 "#PWR049" H 4800 1900 60  0001 C CNN
 F 1 "GND" H 4800 2000 60  0000 C CNN
 F 2 "" H 4800 2150 60  0000 C CNN
@@
 	5150 1650 4800 1650
 $Comp
-L +3V3 #PWR052
+L +3V3 #PWR050
 U 1 1 55055A52
 P 4800 1600
-F 0 "#PWR052" H 4800 1450 60  0001 C CNN
+F 0 "#PWR050" H 4800 1450 60  0001 C CNN
 F 1 "+3V3" H 4800 1740 60  0000 C CNN
 F 2 "" H 4800 1600 60  0000 C CNN
@@
 	4800 1650 4800 1600
 $Comp
-L +3V3 #PWR053
+L +3V3 #PWR051
 U 1 1 55055A97
 P 4400 1500
-F 0 "#PWR053" H 4400 1350 60  0001 C CNN
+F 0 "#PWR051" H 4400 1350 60  0001 C CNN
 F 1 "+3V3" H 4400 1640 60  0000 C CNN
 F 2 "" H 4400 1500 60  0000 C CNN
@@
 	4550 1550 4400 1550
 $Comp
-L GND #PWR054
+L GND #PWR052
 U 1 1 55055AEC
 P 4950 2250
-F 0 "#PWR054" H 4950 2000 60  0001 C CNN
+F 0 "#PWR052" H 4950 2000 60  0001 C CNN
 F 1 "GND" H 4950 2100 60  0000 C CNN
 F 2 "" H 4950 2250 60  0000 C CNN
@@
 $EndComp
 $Comp
-L GND #PWR055
+L GND #PWR053
 U 1 1 55068568
 P 7100 1450
-F 0 "#PWR055" H 7100 1200 60  0001 C CNN
+F 0 "#PWR053" H 7100 1200 60  0001 C CNN
 F 1 "GND" H 7100 1300 60  0000 C CNN
 F 2 "" H 7100 1450 60  0000 C CNN
@@
 	9700 4350 9250 4350
 $Comp
-L GND #PWR056
+L GND #PWR054
 U 1 1 55068D17
 P 9500 4350
-F 0 "#PWR056" H 9500 4100 60  0001 C CNN
+F 0 "#PWR054" H 9500 4100 60  0001 C CNN
 F 1 "GND" H 9500 4200 60  0000 C CNN
 F 2 "" H 9500 4350 60  0000 C CNN
@@
 $EndComp
 $Comp
-L GND #PWR057
+L GND #PWR055
 U 1 1 55068D89
 P 9000 3750
-F 0 "#PWR057" H 9000 3500 60  0001 C CNN
+F 0 "#PWR055" H 9000 3500 60  0001 C CNN
 F 1 "GND" H 9000 3600 60  0000 C CNN
 F 2 "" H 9000 3750 60  0000 C CNN
@@
 Connection ~ 2500 2600
 $Comp
-L +3V3 #PWR058
+L +3V3 #PWR056
 U 1 1 55069C09
 P 2500 2450
-F 0 "#PWR058" H 2500 2300 60  0001 C CNN
+F 0 "#PWR056" H 2500 2300 60  0001 C CNN
 F 1 "+3V3" H 2500 2590 60  0000 C CNN
 F 2 "" H 2500 2450 60  0000 C CNN
@@
 $EndComp
 $Comp
-L GND #PWR059
+L GND #PWR057
 U 1 1 55069C1D
 P 2500 3350
-F 0 "#PWR059" H 2500 3100 60  0001 C CNN
+F 0 "#PWR057" H 2500 3100 60  0001 C CNN
 F 1 "GND" H 2500 3200 60  0000 C CNN
 F 2 "" H 2500 3350 60  0000 C CNN
@@
 $EndComp
 $Comp
-L GND #PWR060
+L GND #PWR058
 U 1 1 5506A4BA
 P 8100 2300
-F 0 "#PWR060" H 8100 2050 60  0001 C CNN
+F 0 "#PWR058" H 8100 2050 60  0001 C CNN
 F 1 "GND" H 8100 2150 60  0000 C CNN
 F 2 "" H 8100 2300 60  0000 C CNN
@@
 Wire Wire Line
 	8100 1750 8100 2300
+Connection ~ 9250 3950
+Connection ~ 9700 3950
+Connection ~ 9500 4350
+Connection ~ 9250 4350
+Connection ~ 9700 4350
 $EndSCHEMATC

Commit message: PCB design
Routing for the main components, except for the power section
Parts:
- TP17, TP18: footprint Measurement_Points:Measurement_Point_Round-SMD-Pad_Small -> Anastasia:Test_Point_Round-SMD-Pad
Connections:
- wire segments 62 -> 63
Changed lines of the file:
@@
 	9950 2800 9950 3950
 Wire Wire Line
-	9950 3950 5150 3950
-Wire Wire Line
-	5150 3950 5150 3000
+	9950 3950 4900 3950
 $Comp
 L C C46
@@
 F 0 "TP17" H 6600 2800 60  0000 C CNN
 F 1 "TESTPAD" H 6400 2600 60  0001 C CNN
-F 2 "Measurement_Points:Measurement_Point_Round-SMD-Pad_Small" H 6600 2800 60  0001 C CNN
+F 2 "Anastasia:Test_Point_Round-SMD-Pad" H 6600 2800 60  0001 C CNN
 F 3 "" H 6600 2800 60  0000 C CNN
 	1    6350 2800
@@
 F 0 "TP18" H 6600 2900 60  0000 C CNN
 F 1 "TESTPAD" H 6400 2700 60  0001 C CNN
-F 2 "Measurement_Points:Measurement_Point_Round-SMD-Pad_Small" H 6600 2900 60  0001 C CNN
+F 2 "Anastasia:Test_Point_Round-SMD-Pad" H 6600 2900 60  0001 C CNN
 F 3 "" H 6600 2900 60  0000 C CNN
 	1    6350 2900
@@
 Connection ~ 9250 4350
 Connection ~ 9700 4350
+Wire Wire Line
+	4900 3950 4900 3000
+Wire Wire Line
+	4900 3000 5150 3000
 $EndSCHEMATC

Commit message: Refactoring
Connections:
- wire segments 63 -> 71
Changed lines of the file:
@@
 LIBS:memory
 LIBS:xilinx
-LIBS:special
 LIBS:microcontrollers
 LIBS:dsp
@@
 U 1 1 550557D1
 P 4050 1500
+AR Path="/550557D1" Ref="C36"  Part="1"
+AR Path="/550556D4/550557D1" Ref="C36"  Part="1"
 F 0 "C36" H 4100 1600 50  0000 L CNN
 F 1 "4.7U" H 4100 1400 50  0000 L CNN
@@
 $EndComp
 Wire Wire Line
-	4050 1300 4050 1150
-Wire Wire Line
-	4050 1850 4050 1700
+	4050 1150 4050 1350
+Wire Wire Line
+	4050 1650 4050 1850
 Wire Wire Line
 	4050 1300 5150 1300
@@
 U 1 1 5505582E
 P 4200 2950
+AR Path="/5505582E" Ref="C41"  Part="1"
+AR Path="/550556D4/5505582E" Ref="C41"  Part="1"
 F 0 "C41" H 4250 3050 50  0000 L CNN
 F 1 "100N" H 4250 2850 50  0000 L CNN
@@
 U 1 1 5505584F
 P 4550 3050
+AR Path="/5505584F" Ref="C43"  Part="1"
+AR Path="/550556D4/5505584F" Ref="C43"  Part="1"
 F 0 "C43" H 4600 3150 50  0000 L CNN
 F 1 "33N" H 4600 2950 50  0000 L CNN
@@
 	4550 2850 5150 2850
 Wire Wire Line
-	5150 2750 4200 2750
-Wire Wire Line
-	4200 3150 4200 3400
+	4200 2750 5150 2750
+Wire Wire Line
+	4200 3100 4200 3400
 Wire Wire Line
 	4200 3400 4550 3400
 Wire Wire Line
-	4550 3400 4550 3250
+	4550 3400 4550 3200
 Connection ~ 4400 3400
 $Comp
@@
 U 1 1 55055963
 P 4400 1750
+AR Path="/55055963" Ref="C37"  Part="1"
+AR Path="/550556D4/55055963" Ref="C37"  Part="1"
 F 0 "C37" H 4450 1850 50  0000 L CNN
 F 1 "100N" H 4450 1650 50  0000 L CNN
@@
 $EndComp
 Wire Wire Line
-	4400 2050 4400 1950
+	4400 1900 4400 2050
 $Comp
 L C C38
 U 1 1 550559C2
 P 4800 1850
+AR Path="/550559C2" Ref="C38"  Part="1"
+AR Path="/550556D4/550559C2" Ref="C38"  Part="1"
 F 0 "C38" H 4850 1950 50  0000 L CNN
 F 1 "1N" H 4850 1750 50  0000 L CNN
@@
 $EndComp
 Wire Wire Line
-	4800 2150 4800 2050
+	4800 2000 4800 2150
 Wire Wire Line
 	5150 1550 5150 1750
@@
 $EndComp
 Wire Wire Line
-	4800 1650 4800 1600
+	4800 1600 4800 1700
 $Comp
 L +3V3 #PWR037
@@
 $EndComp
 Wire Wire Line
-	4400 1550 4400 1500
+	4400 1500 4400 1600
 Wire Wire Line
 	5150 1400 4550 1400
@@
 $EndComp
 Wire Wire Line
-	6250 1450 6400 1450
+	6250 1450 6500 1450
 $Comp
 L INDUCTOR L5
@@
 U 1 1 55068A29
 P 9250 4150
+AR Path="/55068A29" Ref="C46"  Part="1"
+AR Path="/550556D4/55068A29" Ref="C46"  Part="1"
 F 0 "C46" H 9300 4250 50  0000 L CNN
 F 1 "2.2N" H 9300 4050 50  0000 L CNN
@@
 U 1 1 55068B3E
 P 9700 4150
+AR Path="/55068B3E" Ref="C47"  Part="1"
+AR Path="/550556D4/55068B3E" Ref="C47"  Part="1"
 F 0 "C47" H 9750 4250 50  0000 L CNN
 F 1 "N/C" H 9750 4050 50  0000 L CNN
@@
 U 1 1 55068D43
 P 8500 3400
+AR Path="/55068D43" Ref="C44"  Part="1"
+AR Path="/550556D4/55068D43" Ref="C44"  Part="1"
 F 0 "C44" H 8550 3500 50  0000 L CNN
 F 1 "1.8N" H 8550 3300 50  0000 L CNN
@@
 U 1 1 55068D64
 P 8800 3600
+AR Path="/55068D64" Ref="C45"  Part="1"
+AR Path="/550556D4/55068D64" Ref="C45"  Part="1"
 F 0 "C45" H 8850 3700 50  0000 L CNN
 F 1 "1.2N" H 8850 3500 50  0000 L CNN
@@
 	8900 3750 9000 3750
 Wire Wire Line
-	8200 3400 8300 3400
-Wire Wire Line
-	8700 3400 9400 3400
+	8200 3400 8350 3400
+Wire Wire Line
+	8650 3400 9400 3400
 Connection ~ 8800 3400
 Wire Notes Line
@@
 	3100 2600 3250 2600
 Wire Wire Line
-	2500 2450 2500 2850
+	2500 2450 2500 2900
 $Comp
 L C C42
 U 1 1 55069B78
 P 2500 3050
+AR Path="/55069B78" Ref="C42"  Part="1"
+AR Path="/550556D4/55069B78" Ref="C42"  Part="1"
 F 0 "C42" H 2550 3150 50  0000 L CNN
 F 1 "1U" H 2550 2950 50  0000 L CNN
@@
 $EndComp
 Wire Wire Line
-	2500 3350 2500 3250
+	2500 3200 2500 3350
 Text Notes 2650 2450 0    60   ~ 0
 For the internal DC-DC\nLowers power consumption\nCan be avoided in the final design
@@
 U 1 1 5506A386
 P 7900 2050
+AR Path="/5506A386" Ref="C39"  Part="1"
+AR Path="/550556D4/5506A386" Ref="C39"  Part="1"
 F 0 "C39" H 7950 2150 50  0000 L CNN
 F 1 "10P" H 7950 1950 50  0000 L CNN
@@
 U 1 1 5506A3A3
 P 8300 2050
+AR Path="/5506A3A3" Ref="C40"  Part="1"
+AR Path="/550556D4/5506A3A3" Ref="C40"  Part="1"
 F 0 "C40" H 8350 2150 50  0000 L CNN
 F 1 "10P" H 8350 1950 50  0000 L CNN
@@
 $EndComp
 Wire Wire Line
-	7900 2250 7900 2300
+	7900 2200 7900 2300
 Wire Wire Line
 	7900 2300 8300 2300
 Wire Wire Line
-	8300 2300 8300 2250
+	8300 2300 8300 2200
 Connection ~ 8100 2300
 Wire Wire Line
-	8300 1400 8300 1850
-Wire Wire Line
-	7900 1850 7900 1650
+	8300 1400 8300 1900
+Wire Wire Line
+	7900 1650 7900 1900
 Wire Wire Line
 	7900 1650 7450 1650
@@
 Connection ~ 5150 1950
 Wire Wire Line
-	6900 1450 7100 1450
+	6800 1450 7100 1450
 Wire Wire Line
 	8100 1750 8100 2300
@@
 Wire Wire Line
 	4900 3000 5150 3000
+Wire Wire Line
+	4200 2750 4200 2800
+Wire Wire Line
+	4550 2900 4550 2850
+Connection ~ 4800 1650
+Connection ~ 4400 1550
+Connection ~ 4050 1300
+Wire Wire Line
+	8800 3450 8800 3400
+Wire Wire Line
+	8800 3800 8800 3750
+Wire Wire Line
+	9250 4000 9250 3950
+Wire Wire Line
+	9250 4350 9250 4300
+Wire Wire Line
+	9700 4350 9700 4300
+Wire Wire Line
+	9700 4000 9700 3950
 $EndSCHEMATC
