File: KiCad project/Sheet7.sch (KiCad schematic (older format))
At the start: 27 parts, among them U7 AFE4490, X3 CRYSTAL

Commit message: PCB finalised, Gerbers created for v0.5
New footprints, fixes in schematic, PCB final design, plotted Gerbers
for prototype production
Parts:
- D1: footprint (none) -> Anastasia:BPW34S
- D2: footprint (none) -> Resistors_SMD:R_0603_HandSoldering
- D3: footprint (none) -> Anastasia:2x1.25mm_LED
Changed lines of the file:
@@
 $Descr A4 11693 8268
 encoding utf-8
-Sheet 7 10
+Sheet 6 10
 Title "AFE4403"
 Date "17 March 2015"
@@
 	4300 4800 2250 4800
 $Comp
-L GND #PWR032
+L GND #PWR017
 U 1 1 5507E63E
 P 2800 3200
-F 0 "#PWR032" H 2800 2950 60  0001 C CNN
+F 0 "#PWR017" H 2800 2950 60  0001 C CNN
 F 1 "GND" H 2800 3050 60  0000 C CNN
 F 2 "" H 2800 3200 60  0000 C CNN
@@
 $EndComp
 $Comp
-L +3V3 #PWR033
+L +3V3 #PWR018
 U 1 1 5507E9AF
 P 3400 2600
-F 0 "#PWR033" H 3400 2450 60  0001 C CNN
+F 0 "#PWR018" H 3400 2450 60  0001 C CNN
 F 1 "+3V3" H 3400 2740 60  0000 C CNN
 F 2 "" H 3400 2600 60  0000 C CNN
@@
 $EndComp
 $Comp
-L GND #PWR034
+L GND #PWR019
 U 1 1 5507EA5D
 P 4100 3350
-F 0 "#PWR034" H 4100 3100 60  0001 C CNN
+F 0 "#PWR019" H 4100 3100 60  0001 C CNN
 F 1 "GND" H 4100 3200 60  0000 C CNN
 F 2 "" H 4100 3350 60  0000 C CNN
@@
 $EndComp
 $Comp
-L GND #PWR035
+L GND #PWR020
 U 1 1 5507EB22
 P 3400 3050
-F 0 "#PWR035" H 3400 2800 60  0001 C CNN
+F 0 "#PWR020" H 3400 2800 60  0001 C CNN
 F 1 "GND" H 3400 2900 60  0000 C CNN
 F 2 "" H 3400 3050 60  0000 C CNN
@@
 	5150 2600 3400 2600
 $Comp
-L GND #PWR036
+L GND #PWR021
 U 1 1 5507EE1C
 P 1700 2300
-F 0 "#PWR036" H 1700 2050 60  0001 C CNN
+F 0 "#PWR021" H 1700 2050 60  0001 C CNN
 F 1 "GND" H 1700 2150 60  0000 C CNN
 F 2 "" H 1700 2300 60  0000 C CNN
@@
 $EndComp
 $Comp
-L GND #PWR037
+L GND #PWR022
 U 1 1 5507F42E
 P 4700 4600
-F 0 "#PWR037" H 4700 4350 60  0001 C CNN
+F 0 "#PWR022" H 4700 4350 60  0001 C CNN
 F 1 "GND" H 4700 4450 60  0000 C CNN
 F 2 "" H 4700 4600 60  0000 C CNN
@@
 $EndComp
 $Comp
-L +3V3 #PWR038
+L +3V3 #PWR023
 U 1 1 5507F442
 P 4700 4000
-F 0 "#PWR038" H 4700 3850 60  0001 C CNN
+F 0 "#PWR023" H 4700 3850 60  0001 C CNN
 F 1 "+3V3" H 4700 4140 60  0000 C CNN
 F 2 "" H 4700 4000 60  0000 C CNN
@@
 	4700 4100 4700 4000
 $Comp
-L GND #PWR039
+L GND #PWR024
 U 1 1 5507FE0D
 P 3750 3250
-F 0 "#PWR039" H 3750 3000 60  0001 C CNN
+F 0 "#PWR024" H 3750 3000 60  0001 C CNN
 F 1 "GND" H 3750 3100 60  0000 C CNN
 F 2 "" H 3750 3250 60  0000 C CNN
@@
 F 0 "D2" H 2900 4100 50  0000 C CNN
 F 1 "RED_LED" H 2900 3900 50  0000 C CNN
-F 2 "" H 2900 4000 60  0001 C CNN
+F 2 "Resistors_SMD:R_0603_HandSoldering" H 2900 4000 60  0001 C CNN
 F 3 "" H 2900 4000 60  0000 C CNN
 	1    2900 4000
@@
 F 0 "D3" H 2900 4450 50  0000 C CNN
 F 1 "IR_LED" H 2900 4250 50  0000 C CNN
-F 2 "" H 2900 4350 60  0001 C CNN
+F 2 "Anastasia:2x1.25mm_LED" H 2900 4350 60  0001 C CNN
 F 3 "" H 2900 4350 60  0000 C CNN
 	1    2900 4350
@@
 F 0 "D1" H 2500 1200 50  0000 C CNN
 F 1 "PHOTODIODE" H 2500 1000 50  0000 C CNN
-F 2 "" H 2500 1100 60  0001 C CNN
+F 2 "Anastasia:BPW34S" H 2500 1100 60  0001 C CNN
 F 3 "" H 2500 1100 60  0000 C CNN
 	1    2500 1100
@@
 Connection ~ 8850 1700
 $Comp
-L +3V3 #PWR040
+L +3V3 #PWR025
 U 1 1 55080B5C
 P 8850 1050
-F 0 "#PWR040" H 8850 900 60  0001 C CNN
+F 0 "#PWR025" H 8850 900 60  0001 C CNN
 F 1 "+3V3" H 8850 1190 60  0000 C CNN
 F 2 "" H 8850 1050 60  0000 C CNN
@@
 $EndComp
 $Comp
-L +3V3 #PWR041
+L +3V3 #PWR026
 U 1 1 550D77E4
 P 700 1750
-F 0 "#PWR041" H 700 1600 60  0001 C CNN
+F 0 "#PWR026" H 700 1600 60  0001 C CNN
 F 1 "+3V3" H 700 1890 60  0000 C CNN
 F 2 "" H 700 1750 60  0000 C CNN
@@
 Connection ~ 5150 2000
 $Comp
-L GND #PWR042
+L GND #PWR027
 U 1 1 550F0F16
 P 4800 2000
-F 0 "#PWR042" H 4800 1750 60  0001 C CNN
+F 0 "#PWR027" H 4800 1750 60  0001 C CNN
 F 1 "GND" H 4800 1850 60  0000 C CNN
 F 2 "" H 4800 2000 60  0000 C CNN
@@
 	5050 3100 5150 3100
 $Comp
-L +3V3 #PWR043
+L +3V3 #PWR028
 U 1 1 550F38B0
 P 4800 3100
-F 0 "#PWR043" H 4800 2950 60  0001 C CNN
+F 0 "#PWR028" H 4800 2950 60  0001 C CNN
 F 1 "+3V3" H 4800 3240 60  0000 C CNN
 F 2 "" H 4800 3100 60  0000 C CNN
@@
 	4700 3050 4600 3050
 $Comp
-L GND #PWR044
+L GND #PWR029
 U 1 1 550F3EF5
 P 4850 3350
-F 0 "#PWR044" H 4850 3100 60  0001 C CNN
+F 0 "#PWR029" H 4850 3100 60  0001 C CNN
 F 1 "GND" H 4850 3200 60  0000 C CNN
 F 2 "" H 4850 3350 60  0000 C CNN

Commit message: Refactoring
Parts:
- C30, C31, C32: value 0.1U -> 100N
- C34, C35: value C -> 10P
Connections:
- wire segments 89 -> 101
Other:
- note added: "Analog supply \ndecoupling\nand anti-EMF"
Changed lines of the file:
@@
 LIBS:memory
 LIBS:xilinx
-LIBS:special
 LIBS:microcontrollers
 LIBS:dsp
@@
 L GND #PWR017
 U 1 1 5507E63E
-P 2800 3200
-F 0 "#PWR017" H 2800 2950 60  0001 C CNN
-F 1 "GND" H 2800 3050 60  0000 C CNN
-F 2 "" H 2800 3200 60  0000 C CNN
-F 3 "" H 2800 3200 60  0000 C CNN
-	1    2800 3200
+P 2800 3100
+F 0 "#PWR017" H 2800 2850 60  0001 C CNN
+F 1 "GND" H 2800 2950 60  0000 C CNN
+F 2 "" H 2800 3100 60  0000 C CNN
+F 3 "" H 2800 3100 60  0000 C CNN
+	1    2800 3100
 	-1   0    0    -1
 $EndComp
@@
 U 1 1 5507E652
 P 3000 2850
+AR Path="/5507E652" Ref="C34"  Part="1"
+AR Path="/5507E4D4/5507E652" Ref="C34"  Part="1"
 F 0 "C34" H 3050 2950 50  0000 L CNN
-F 1 "C" H 3050 2750 50  0000 L CNN
+F 1 "10P" H 3050 2750 50  0000 L CNN
 F 2 "Capacitors_SMD:C_0603" H 3038 2700 30  0001 C CNN
 F 3 "" H 3000 2850 60  0000 C CNN
@@
 U 1 1 5507E675
 P 2600 2750
+AR Path="/5507E675" Ref="C35"  Part="1"
+AR Path="/5507E4D4/5507E675" Ref="C35"  Part="1"
 F 0 "C35" H 2650 2850 50  0000 L CNN
-F 1 "C" H 2650 2650 50  0000 L CNN
+F 1 "10P" H 2650 2650 50  0000 L CNN
 F 2 "Capacitors_SMD:C_0603" H 2638 2600 30  0001 C CNN
 F 3 "" H 2600 2750 60  0000 C CNN
@@
 U 1 1 5507EA21
 P 4100 3050
+AR Path="/5507EA21" Ref="C33"  Part="1"
+AR Path="/5507E4D4/5507EA21" Ref="C33"  Part="1"
 F 0 "C33" H 4150 3150 50  0000 L CNN
 F 1 "2.2U" H 4150 2950 50  0000 L CNN
@@
 U 1 1 5507EAF1
 P 3400 2800
+AR Path="/5507EAF1" Ref="C31"  Part="1"
+AR Path="/5507E4D4/5507EAF1" Ref="C31"  Part="1"
 F 0 "C31" H 3450 2900 50  0000 L CNN
-F 1 "0.1U" H 3450 2700 50  0000 L CNN
+F 1 "100N" H 3450 2700 50  0000 L CNN
 F 2 "Capacitors_SMD:C_0603" H 3438 2650 30  0001 C CNN
 F 3 "" H 3400 2800 60  0000 C CNN
@@
 	3300 2250 2600 2250
 Wire Wire Line
-	2600 2250 2600 2550
+	2600 2250 2600 2600
 Connection ~ 2600 2400
 Wire Wire Line
-	3000 3100 3000 3050
-Wire Wire Line
-	2600 3100 2800 3200
-Wire Wire Line
-	2800 3200 3000 3100
-Wire Wire Line
-	2600 3100 2600 2950
-Connection ~ 2800 3200
-Wire Wire Line
-	4100 3350 4100 3250
-Wire Wire Line
-	3400 3050 3400 3000
+	3000 3100 3000 3000
+Wire Wire Line
+	2600 3100 3000 3100
+Wire Wire Line
+	2600 2900 2600 3100
+Connection ~ 2800 3100
+Wire Wire Line
+	4100 3200 4100 3350
+Wire Wire Line
+	3400 2950 3400 3050
 Wire Wire Line
 	5150 2600 3400 2600
@@
 U 1 1 5507EE30
 P 1950 2100
+AR Path="/5507EE30" Ref="C30"  Part="1"
+AR Path="/5507E4D4/5507EE30" Ref="C30"  Part="1"
 F 0 "C30" H 2000 2200 50  0000 L CNN
-F 1 "0.1U" H 2000 2000 50  0000 L CNN
+F 1 "100N" H 2000 2000 50  0000 L CNN
 F 2 "Capacitors_SMD:C_0603" H 1988 1950 30  0001 C CNN
 F 3 "" H 1950 2100 60  0000 C CNN
@@
 U 1 1 5507F407
 P 4700 4300
+AR Path="/5507F407" Ref="C26"  Part="1"
+AR Path="/5507E4D4/5507F407" Ref="C26"  Part="1"
 F 0 "C26" H 4750 4400 50  0000 L CNN
 F 1 "1U" H 4750 4200 50  0000 L CNN
@@
 $EndComp
 Wire Wire Line
-	4700 4600 4700 4500
-Wire Wire Line
-	4700 4100 4700 4000
+	4700 4450 4700 4600
+Wire Wire Line
+	4700 4000 4700 4150
 $Comp
 L GND #PWR024
@@
 U 1 1 5507FE21
 P 3750 3000
+AR Path="/5507FE21" Ref="C27"  Part="1"
+AR Path="/5507E4D4/5507FE21" Ref="C27"  Part="1"
 F 0 "C27" H 3800 3100 50  0000 L CNN
 F 1 "2.2U" H 3800 2900 50  0000 L CNN
@@
 $EndComp
 Wire Wire Line
-	3750 3250 3750 3200
+	3750 3150 3750 3250
 Wire Wire Line
 	3750 2800 5150 2800
@@
 $EndComp
 Wire Wire Line
-	8850 1200 8850 1050
+	8850 1050 8850 1300
 $Comp
 L C C28
 U 1 1 550D75B9
 P 2500 2100
+AR Path="/550D75B9" Ref="C28"  Part="1"
+AR Path="/5507E4D4/550D75B9" Ref="C28"  Part="1"
 F 0 "C28" H 2550 2200 50  0000 L CNN
 F 1 "10N" H 2550 2000 50  0000 L CNN
@@
 U 1 1 550D75A0
 P 2250 2100
+AR Path="/550D75A0" Ref="C29"  Part="1"
+AR Path="/5507E4D4/550D75A0" Ref="C29"  Part="1"
 F 0 "C29" H 2300 2200 50  0000 L CNN
 F 1 "10N" H 2300 2000 50  0000 L CNN
@@
 U 1 1 550F3E12
 P 4600 3250
+AR Path="/550F3E12" Ref="C32"  Part="1"
+AR Path="/5507E4D4/550F3E12" Ref="C32"  Part="1"
 F 0 "C32" H 4650 3350 50  0000 L CNN
-F 1 "0.1U" H 4650 3150 50  0000 L CNN
+F 1 "100N" H 4650 3150 50  0000 L CNN
 F 2 "Capacitors_SMD:C_0603" H 4638 3100 30  0001 C CNN
 F 3 "" H 4600 3250 60  0000 C CNN
@@
 Connection ~ 2250 1900
 Connection ~ 5150 4100
+Wire Wire Line
+	1950 1950 1950 1900
+Wire Wire Line
+	2250 1950 2250 1900
+Wire Wire Line
+	2500 1950 2500 1900
+Wire Wire Line
+	2500 2300 2500 2250
+Wire Wire Line
+	2250 2300 2250 2250
+Wire Wire Line
+	1950 2250 1950 2300
+Wire Wire Line
+	3000 2700 3000 2650
+Wire Wire Line
+	3400 2600 3400 2650
+Connection ~ 3400 3000
+Wire Wire Line
+	3750 2850 3750 2800
+Wire Wire Line
+	4100 2900 4100 2850
+Connection ~ 4100 3250
+Wire Wire Line
+	4600 3450 4600 3400
+Wire Wire Line
+	4600 3050 4600 3100
+Connection ~ 4700 4100
+Connection ~ 4700 4500
+Wire Wire Line
+	8850 1700 8850 1600
+Text Notes 900  2350 0    60   ~ 0
+Analog supply \ndecoupling\nand anti-EMF
 $EndSCHEMATC
