File: KiCad project/Sheet8.sch (KiCad schematic (older format))
At the start: 1 part, among them U1 EFM32GG332

Commit message: PCB design
Routing for the main components, except for the power section
Connections:
- net PC6 is gone; now on net I2C0_SDA: U1.37 (PC6_/_ACMP0_CH6_/_ETM_TCLK_#2_/_I2C0_SDA_#2_/_LES_CH6_/_LEU1_TX_#0)
- net I2C0_SCL: now also U1.38 (PC7_/_ACMP0_CH7_/_ETM_TD0_#2_/_I2C0_SCL_#2_/_LES_CH7_/_LEU1_RX); no longer U1.35 (PD7_/_ACMP1_O_#2_/_ADC0_CH7_/_CMU_CLK0_#2_/_DAC0_N1/OPAMP_N1_/_ETM_TCLK_#0_/_I2C0_SCL_#1_/_LES_ALTEX1_/_LETIM0_OUT1_#0_/_PCNT0_S1IN_#3_/_TIM1_CC1_#4_/_US1_TX_#2)
- net I2C0_SDA: no longer U1.34 (PD6_/_ACMP0_O_#2_/_ADC0_CH6_/_DAC0_P1/OPAMP_P1_/_ETM_TD0_#0_/_I2C0_SDA_#1_/_LES_ALTEX0_/_LETIM0_OUT0_#0_/_PCNT0_S0IN_#3_/_TIM1_CC0_#4_/_US1_RX_#2)
- new net PD6: U1.34 (PD6_/_ACMP0_O_#2_/_ADC0_CH6_/_DAC0_P1/OPAMP_P1_/_ETM_TD0_#0_/_I2C0_SDA_#1_/_LES_ALTEX0_/_LETIM0_OUT0_#0_/_PCNT0_S0IN_#3_/_TIM1_CC0_#4_/_US1_RX_#2)
- new net PD7: U1.35 (PD7_/_ACMP1_O_#2_/_ADC0_CH7_/_CMU_CLK0_#2_/_DAC0_N1/OPAMP_N1_/_ETM_TCLK_#0_/_I2C0_SCL_#1_/_LES_ALTEX1_/_LETIM0_OUT1_#0_/_PCNT0_S1IN_#3_/_TIM1_CC1_#4_/_US1_TX_#2)
Changed lines of the file:
@@
 Text HLabel 2650 1650 0    60   3State ~ 0
 I2C1_SCL
-Text HLabel 2650 3150 0    60   3State ~ 0
+Text HLabel 2650 1750 0    60   3State ~ 0
 I2C0_SDA
-Text HLabel 2650 3250 0    60   3State ~ 0
+Text HLabel 2650 1850 0    60   3State ~ 0
 I2C0_SCL
 Wire Wire Line
@@
 	2800 1650 2650 1650
 Wire Wire Line
-	2650 3150 2800 3150
+	2650 1750 2800 1750
 Wire Wire Line
-	2650 3250 2800 3250
+	2650 1850 2800 1850
 Text HLabel 2650 2550 0    60   3State ~ 0
 US1_TX
@@
 Text HLabel 1650 3350 0    60   3State ~ 0
 PD8
-Text HLabel 1650 1750 0    60   3State ~ 0
-PC6
 Wire Wire Line
 	2800 3350 1650 3350
+Text HLabel 2600 3150 0    60   BiDi ~ 0
+PD6
+Text HLabel 2600 3250 0    60   BiDi ~ 0
+PD7
 Wire Wire Line
-	1650 1750 2800 1750
+	2800 3150 2600 3150
+Wire Wire Line
+	2600 3250 2800 3250
 $EndSCHEMATC

Commit message: PCB finalised, Gerbers created for v0.5
New footprints, fixes in schematic, PCB final design, plotted Gerbers
for prototype production
Parts:
- added SW1, SW2, SW3: SWITCH, Anastasia:KMS_SMD_SW, symbol SWITCH
Connections:
- net at U1.11 (PC2_/_ACMP0_CH2_/_DAC0_OUT0ALT/OPAMP_OUT0ALT_#2_/_LES_CH2_/_TIM0_CDTI0_#4_/_US2_TX): now also SW1.3
- net at U1.9 (PC0_/_ACMP0_CH0_/_DAC0_OUT0ALT/OPAMP_OUT0ALT_#0_/_I2C0_SDA_#4_/_LES_CH0_/_PCNT0_S0IN_#2_/_PRS_CH2_#0_/_TIM0_CC1_#4_/_US0_TX_#5_/_US1_TX_#0): now also SW3.1
- net PC3: no longer names the net of U1.12 (PC3_/_ACMP0_CH3_/_DAC0_OUT0ALT/OPAMP_OUT0ALT_#3_/_LES_CH3_/_TIM0_CDTI1_#4_/_US2_RX)
- net PC3: now also SW2.1
- new net GND: SW1.2, SW2.4, SW3.4
Changed lines of the file:
@@
 $Descr A4 11693 8268
 encoding utf-8
-Sheet 8 10
+Sheet 7 10
 Title "uC part B"
 Date "17 March 2015"
@@
 Wire Wire Line
 	2800 3050 1900 3050
-Text HLabel 2150 1450 0    60   3State ~ 0
-PC3
-Wire Wire Line
-	2150 1450 2800 1450
 Text HLabel 1650 3350 0    60   3State ~ 0
 PD8
@@
 Wire Wire Line
 	2600 3250 2800 3250
+Wire Wire Line
+	2150 1150 2800 1150
+$Comp
+L SWITCH SW3
+U 1 1 552132DD
+P 1450 950
+F 0 "SW3" H 1450 1050 50  0000 C CNN
+F 1 "SWITCH" H 1450 850 50  0000 C CNN
+F 2 "Anastasia:KMS_SMD_SW" H 1450 950 60  0001 C CNN
+F 3 "" H 1450 950 60  0000 C CNN
+	1    1450 950
+	-1   0    0    -1
+$EndComp
+$Comp
+L SWITCH SW1
+U 1 1 552132FE
+P 1450 1300
+F 0 "SW1" H 1450 1400 50  0000 C CNN
+F 1 "SWITCH" H 1450 1200 50  0000 C CNN
+F 2 "Anastasia:KMS_SMD_SW" H 1450 1300 60  0001 C CNN
+F 3 "" H 1450 1300 60  0000 C CNN
+	1    1450 1300
+	-1   0    0    -1
+$EndComp
+$Comp
+L SWITCH SW2
+U 1 1 55213389
+P 1450 1650
+F 0 "SW2" H 1450 1750 50  0000 C CNN
+F 1 "SWITCH" H 1450 1550 50  0000 C CNN
+F 2 "Anastasia:KMS_SMD_SW" H 1450 1650 60  0001 C CNN
+F 3 "" H 1450 1650 60  0000 C CNN
+	1    1450 1650
+	-1   0    0    -1
+$EndComp
+Wire Wire Line
+	2050 1350 2800 1350
+Wire Wire Line
+	2100 1450 2800 1450
+$Comp
+L GND #PWR030
+U 1 1 5521388B
+P 650 1350
+F 0 "#PWR030" H 650 1100 60  0001 C CNN
+F 1 "GND" H 650 1200 60  0000 C CNN
+F 2 "" H 650 1350 60  0000 C CNN
+F 3 "" H 650 1350 60  0000 C CNN
+	1    650  1350
+	1    0    0    -1
+$EndComp
+Wire Wire Line
+	650  1300 650  1350
+Wire Wire Line
+	650  1300 950  1300
+Wire Wire Line
+	800  1100 800  1800
+Connection ~ 800  1300
+Wire Wire Line
+	2100 1450 2100 1650
+Wire Wire Line
+	2100 1650 1950 1650
+Wire Wire Line
+	2150 1150 2150 950
+Wire Wire Line
+	2150 950  1950 950
+Wire Wire Line
+	1950 1450 2050 1450
+Wire Wire Line
+	2050 1450 2050 1350
+Wire Wire Line
+	800  1800 950  1800
+Wire Wire Line
+	950  1100 800  1100
 $EndSCHEMATC
