File: KiCad project/Sheet9.sch (KiCad schematic (older format))
At the start: 1 part, among them U1 EFM32GG332

Commit message: PCB design
Routing for the main components, except for the power section
Connections:
- net PF2: now reaches U1.51 (PF2_/_ACMP1_O_#0_/_DBG_SWO_#0_/_GPIO_EM4WU4_/_LEU0_TX_#4_/_TIM0_CC2_#5)
Changed lines of the file:
@@
 Wire Wire Line
 	5250 2800 5400 2800
+Text HLabel 5200 2900 0    60   3State ~ 0
+PF2
+Wire Wire Line
+	5200 2900 5400 2900
 $EndSCHEMATC

Commit message: PCB finalised, Gerbers created for v0.5
New footprints, fixes in schematic, PCB final design, plotted Gerbers
for prototype production
Connections:
- net PE8: now reaches U1.57 (PE8_/_PCNT2_S0IN_#1_/_PRS_CH3_#1)
- net PE9: now reaches U1.58 (PE9_/_PCNT2_S1IN_#1)
Changed lines of the file:
@@
 $Descr A4 11693 8268
 encoding utf-8
-Sheet 9 10
+Sheet 8 10
 Title "uC part C"
 Date "17 March 2015"
@@
 Wire Wire Line
 	5200 2900 5400 2900
+Text HLabel 5250 1850 0    60   3State ~ 0
+PE9
+Wire Wire Line
+	5400 1850 5250 1850
+Text HLabel 5250 1750 0    60   3State ~ 0
+PE8
+Wire Wire Line
+	5400 1750 5250 1750
 $EndSCHEMATC
